File: greenenergyecu/greenenergyecu.kicad_pcb (KiCad board)
At the start: 2 copper layers, 34.5 x 20.5 mm, 1 part, among them U1 ICM7555xB

Commit message: yu
Parts:
- moved U1 91.7 mm to (19.0, 9.13)
Routing:
- net (no net): vias 0 -> 5
Changed lines of the file:
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@@
 	(footprint "Package_SO:SOIC-8_3.9x4.9mm_P1.27mm"
 		(layer "F.Cu")
-		(at 87.525 70.095)
+		(at 19.025 9.135)
 		(descr "SOIC, 8 Pin (JEDEC MS-012AA, https://www.analog.com/media/en/package-pcb-resources/package/pkg_pdf/soic_narrow-r/r_8.pdf), generated with kicad-footprint-generator ipc_gullwing_generator.py")
 		(tags "SOIC SO")
@@
 	)
 	(gr_rect
-		(start 68.5 61)
-		(end 103 81.5)
+		(start 0 0.04)
+		(end 34.5 20.54)
 		(stroke
 			(width 0.05)
@@
 		(layer "Edge.Cuts")
 	)
-	(segment
-		(start 85.05 69.46)
-		(end 86.024999 69.46)
-		(width 0.2)
-		(layer "F.Cu")
-		(net 7)
-	)
-	(segment
-		(start 92 68)
-		(end 91.81 68.19)
-		(width 0.2)
-		(layer "F.Cu")
-		(net 7)
-	)
-	(segment
-		(start 88.984999 66.5)
-		(end 92 66.5)
-		(width 0.2)
-		(layer "F.Cu")
-		(net 7)
-	)
-	(segment
-		(start 92 66.5)
-		(end 92 68)
-		(width 0.2)
-		(layer "F.Cu")
-		(net 7)
-	)
-	(segment
-		(start 86.024999 69.46)
-		(end 88.984999 66.5)
-		(width 0.2)
-		(layer "F.Cu")
-		(net 7)
-	)
-	(segment
-		(start 91.81 68.19)
-		(end 90 68.19)
-		(width 0.2)
-		(layer "F.Cu")
+	(via
+		(at 1 1.04)
+		(size 0.6)
+		(drill 0.3)
+		(layers "F.Cu" "B.Cu")
+		(net 0)
+	)
+	(via
+		(at 0 0.04)
+		(size 0.6)
+		(drill 0.3)
+		(layers "F.Cu" "B.Cu")
+		(net 0)
+	)
+	(via
+		(at 1.5 19.04)
+		(size 0.6)
+		(drill 0.3)
+		(layers "F.Cu" "B.Cu")
+		(net 0)
+	)
+	(via
+		(at 33 19.04)
+		(size 0.6)
+		(drill 0.3)
+		(layers "F.Cu" "B.Cu")
+		(net 0)
+	)
+	(via
+		(at 33 1.54)
+		(size 0.6)
+		(drill 0.3)
+		(layers "F.Cu" "B.Cu")
+		(net 0)
+	)
+	(segment
+		(start 16.55 8.5)
+		(end 17.524999 8.5)
+		(width 0.2)
+		(layer "F.Cu")
+		(net 7)
+	)
+	(segment
+		(start 23.5 7.04)
+		(end 23.31 7.23)
+		(width 0.2)
+		(layer "F.Cu")
+		(net 7)
+	)
+	(segment
+		(start 20.484999 5.54)
+		(end 23.5 5.54)
+		(width 0.2)
+		(layer "F.Cu")
+		(net 7)
+	)
+	(segment
+		(start 23.5 5.54)
+		(end 23.5 7.04)
+		(width 0.2)
+		(layer "F.Cu")
+		(net 7)
+	)
+	(segment
+		(start 17.524999 8.5)
+		(end 20.484999 5.54)
+		(width 0.2)
+		(layer "F.Cu")
+		(net 7)
+	)
+	(segment
+		(start 23.31 7.23)
+		(end 21.5 7.23)
+		(width 0.2)
+		(layer "F.Cu")
