File: greenenergyecu.kicad_pcb (KiCad board)
At the start: 2 copper layers, 34.5 x 20.5 mm, 1 part, among them M2 Module-knock-0.2

Commit message: ssamklms
Parts:
- added M1: Module-vr-discrete-0.5, hellen-one-vr-discrete-0.5:vr-discrete, F.Cu at (7.53, 18.3)
Connections:
- M2 pad W1: unconnected-(M2-IN_KNOCK-PadW1) -> Net-(M1-OUT)
Routing:
- net Net-(M1-OUT): track 0.00 -> 27.7 mm

Commit message: gwvqjehqdwlj
Parts:
- added M3: Module-vr-0.1, hellen-one-vr-0.1:vr, F.Cu at (12.3, 19.9)
- moved M2 11.4 mm to (21.9, 5.74)
- moved M1 9.26 mm to (2.34, 10.6)
Connections:
- M2 pad E3: unconnected-(M2-OUT_KNOCK-PadE3) -> Net-(M2-OUT_KNOCK)
Routing:
- net Net-(M1-OUT): track 27.7 -> 5.63 mm
- net Net-(M2-OUT_KNOCK): track 0.00 -> 12.5 mm

Commit message: wew
Parts:
- added M4: Module-motor-driver-0.1, motor-driver:motor-driver, F.Cu at (8.66, -0.69)
Routing:
- net (no net): vias 5 -> 3
Other:
- board size 34.5 x 20.5 mm -> 34.5 x 35.2 mm

Commit message: wew
Parts:
- moved M4 13.6 mm to (10.1, -14.2), turned to -90 degrees
- moved M3 12.2 mm to (0.02, 20.4)
Routing:
- net (no net): vias 3 -> 2
Changed lines of the file:
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@@
 	(footprint "motor-driver:motor-driver"
 		(layer "F.Cu")
-		(at 8.66 -0.69)
+		(at 10.105 -14.205 -90)
 		(property "Reference" "M4"
-			(at 2.45 -9.8 0)
+			(at 2.45 -9.8 -90)
 			(unlocked yes)
 			(layer "F.SilkS")
@@
 		)
 		(property "Value" "Module-motor-driver-0.1"
-			(at 9.4 -11.3 0)
+			(at 9.4 -11.3 -90)
 			(unlocked yes)
 			(layer "F.Fab")
@@
 		)
 		(property "Footprint" "motor-driver:motor-driver"
-			(at 0 0 0)
+			(at 0 0 90)
 			(layer "F.Fab")
 			(hide yes)
@@
 		)
 		(property "Datasheet" ""
-			(at 0 0 0)
+			(at 0 0 90)
 			(layer "F.Fab")
 			(hide yes)
@@
 		)
 		(property "Description" ""
-			(at 0 0 0)
+			(at 0 0 90)
 			(layer "F.Fab")
 			(hide yes)
@@
 		)
 		(pad "G" smd rect
-			(at 0.1 -2.2 180)
+			(at 0.1 -2.2 90)
 			(size 0.2 4.4)
 			(layers "F.Cu")
@@
 		)
 		(pad "G" smd rect
-			(at 0.1 -2.2 180)
+			(at 0.1 -2.2 90)
 			(size 0.2 4.4)
 			(layers "In1.Cu")
@@
 		)
 		(pad "G" smd rect
-			(at 0.1 -2.2 180)
+			(at 0.1 -2.2 90)
 			(size 0.2 4.4)
 			(layers "In2.Cu")
@@
 		)
 		(pad "G" smd rect
-			(at 0.1 -2.2 180)
+			(at 0.1 -2.2 90)
 			(size 0.2 4.4)
 			(layers "B.Cu")
@@
 		)
 		(pad "G" smd rect
-			(at 0.6 -0.1 270)
+			(at 0.6 -0.1 180)
 			(size 0.2 1.2)
 			(layers "F.Cu")
@@
 		)
 		(pad "G" smd rect
-			(at 0.6 -0.1 270)
+			(at 0.6 -0.1 180)
 			(size 0.2 1.2)
 			(layers "In1.Cu")
@@
 		)
 		(pad "G" smd rect
-			(at 0.6 -0.1 270)
+			(at 0.6 -0.1 180)
 			(size 0.2 1.2)
 			(layers "In2.Cu")
@@
 		)
 		(pad "G" smd rect
-			(at 0.6 -0.1 270)
+			(at 0.6 -0.1 180)
 			(size 0.2 1.2)
 			(layers "B.Cu")
@@
 		)
 		(pad "G" smd rect
-			(at 5 -9.9 270)
+			(at 5 -9.9 180)
 			(size 0.2 6.8)
 			(layers "F.Cu")
@@
 		)
 		(pad "G" smd rect
-			(at 5 -9.9 270)
+			(at 5 -9.9 180)
 			(size 0.2 6.8)
 			(layers "In1.Cu")
@@
 		)
 		(pad "G" smd rect
-			(at 5 -9.9 270)
+			(at 5 -9.9 180)
 			(size 0.2 6.8)
 			(layers "In2.Cu")
@@
 		)
 		(pad "G" smd rect
-			(at 5 -9.9 270)
+			(at 5 -9.9 180)
 			(size 0.2 6.8)
 			(layers "B.Cu")
@@
 		)
 		(pad "G" smd rect
-			(at 7.2 -0.1 270)
+			(at 7.2 -0.1 180)
 			(size 0.2 6.8)
 			(layers "F.Cu")
@@
 		)
 		(pad "G" smd rect
-			(at 7.2 -0.1 270)
+			(at 7.2 -0.1 180)
 			(size 0.2 6.8)
 			(layers "In1.Cu")
@@
 		)
 		(pad "G" smd rect
-			(at 7.2 -0.1 270)
+			(at 7.2 -0.1 180)
 			(size 0.2 6.8)
 			(layers "In2.Cu")
@@
 		)
 		(pad "G" smd rect
-			(at 7.2 -0.1 270)
+			(at 7.2 -0.1 180)
 			(size 0.2 6.8)
 			(layers "B.Cu")
@@
 		)
 		(pad "G" smd rect
-			(at 11.8 -9.9 270)
+			(at 11.8 -9.9 180)
 			(size 0.2 4)
 			(layers "F.Cu")
@@
 		)
 		(pad "G" smd rect
-			(at 11.8 -9.9 270)
+			(at 11.8 -9.9 180)
 			(size 0.2 4)
 			(layers "In1.Cu")
@@
 		)
 		(pad "G" smd rect
-			(at 11.8 -9.9 270)
+			(at 11.8 -9.9 180)
 			(size 0.2 4)
 			(layers "In2.Cu")
@@
 		)
 		(pad "G" smd rect
-			(at 11.8 -9.9 270)
+			(at 11.8 -9.9 180)
 			(size 0.2 4)
 			(layers "B.Cu")
@@
 		)
 		(pad "G" smd rect
-			(at 12.9 -0.1 270)
+			(at 12.9 -0.1 180)
 			(size 0.2 1.8)
 			(layers "F.Cu")
@@
 		)
 		(pad "G" smd rect
-			(at 12.9 -0.1 270)
+			(at 12.9 -0.1 180)
 			(size 0.2 1.8)
 			(layers "In1.Cu")
@@
 		)
 		(pad "G" smd rect
-			(at 12.9 -0.1 270)
+			(at 12.9 -0.1 180)
 			(size 0.2 1.8)
 			(layers "In2.Cu")
@@
 		)
 		(pad "G" smd rect
-			(at 12.9 -0.1 270)
+			(at 12.9 -0.1 180)
 			(size 0.2 1.8)
 			(layers "B.Cu")
@@
 		)
 		(pad "G" smd rect
-			(at 13.7 -5 180)
+			(at 13.7 -5 90)
 			(size 0.2 10)
 			(layers "F.Cu")
@@
 		)
 		(pad "G" smd rect
-			(at 13.7 -5 180)
+			(at 13.7 -5 90)
 			(size 0.2 10)
 			(layers "In1.Cu")
@@
 		)
 		(pad "G" smd rect
-			(at 13.7 -5 180)
+			(at 13.7 -5 90)
 			(size 0.2 10)
 			(layers "In2.Cu")
@@
 		)
 		(pad "G" smd rect
-			(at 13.7 -5 180)
+			(at 13.7 -5 90)
 			(size 0.2 10)
 			(layers "B.Cu")
@@
 		)
 		(pad "N1" thru_hole circle
-			(at 1.1 -9.7 90)
+			(at 1.1 -9.7)
 			(size 0.6 0.6)
 			(drill 0.3)
@@
 		)
 		(pad "N2" thru_hole circle
-			(at 9.1 -9.5 180)
+			(at 9.1 -9.5 90)
 			(size 1 1)
 			(drill 0.7)
@@
 		)
 		(pad "S1" thru_hole circle
-			(at 1.9 -0.5 180)
+			(at 1.9 -0.5 90)
 			(size 1 1)
 			(drill 0.7)
@@
 		)
 		(pad "S2" thru_hole circle
-			(at 3.1 -0.5 180)
+			(at 3.1 -0.5 90)
 			(size 1 1)
 			(drill 0.7)
@@
 		)
 		(pad "S3" thru_hole circle
-			(at 11.3 -0.5 180)
+			(at 11.3 -0.5 90)
 			(size 1 1)
 			(drill 0.7)
@@
 		)
 		(pad "W1" thru_hole circle
-			(at 0.3 -9.7 90)
+			(at 0.3 -9.7)
 			(size 0.6 0.6)
 			(drill 0.3)
@@
 		)
 		(pad "W2" thru_hole circle
-			(at 0.3 -8.9 90)
+			(at 0.3 -8.9)
 			(size 0.6 0.6)
 			(drill 0.3)
@@
 		)
 		(pad "W3" thru_hole circle
-			(at 0.3 -8.1 90)
+			(at 0.3 -8.1)
 			(size 0.6 0.6)
 			(drill 0.3)
@@
 		)
 		(pad "W4" thru_hole circle
-			(at 0.3 -7.3 90)
+			(at 0.3 -7.3)
 			(size 0.6 0.6)
 			(drill 0.3)
@@
 		)
 		(pad "W5" thru_hole circle
-			(at 0.3 -6.5 90)
+			(at 0.3 -6.5)
 			(size 0.6 0.6)
 			(drill 0.3)
@@
 		)
 		(pad "W6" thru_hole circle
-			(at 0.3 -5.7 90)
+			(at 0.3 -5.7)
 			(size 0.6 0.6)
 			(drill 0.3)
@@
 		)
 		(pad "W7" thru_hole circle
-			(at 0.3 -4.9 90)
+			(at 0.3 -4.9)
 			(size 0.6 0.6)
 			(drill 0.3)
@@
 			(polygon
 				(pts
-					(xy 22.36 -0.79) (xy 8.76 -0.79) (xy 8.76 -10.59) (xy 22.36 -10.59)
+					(xy 10.205 -0.505) (xy 10.205 -14.105) (xy 20.005 -14.105) (xy 20.005 -0.505)
 				)
 			)
@@
 	(footprint "hellen-one-vr-0.1:vr"
 		(layer "F.Cu")
-		(at 12.250002 19.89)
+		(at 0.015876 20.388602)
 		(property "Reference" "M3"
 			(at 0.0762 -9.017 0)
@@
 			(polygon
 				(pts
-					(xy 12.67726 19.665) (xy 12.67726 18.768986) (xy 12.474467 18.768986) (xy 12.275002 18.768986)
-					(xy 12.275002 11.915) (xy 12.847867 11.633171) (xy 12.994849 11.940003) (xy 17.993204 11.940003)
-					(xy 18.19284 11.633171) (xy 18.762044 11.633171) (xy 18.888074 11.940003) (xy 32.15 11.939957)
-					(xy 32.15 19.665)
+					(xy 0.443134 20.163602) (xy 0.443134 19.267588) (xy 0.240341 19.267588) (xy 0.040876 19.267588)
+					(xy 0.040876 12.413602) (xy 0.613741 12.131773) (xy 0.760723 12.438605) (xy 5.759078 12.438605)
+					(xy 5.958714 12.131773) (xy 6.527918 12.131773) (xy 6.653948 12.438605) (xy 19.915874 12.438559)
+					(xy 19.915874 20.163602)
 				)
 			)
@@
 	)
 	(via
-		(at 1.5 19.04)
-		(size 0.6)
-		(drill 0.3)
-		(layers "F.Cu" "B.Cu")
-		(net 0)
-	)
-	(via
